Commit message: change: LRF pose for custom robot

File: urdf/minibot_light_01.xacro (robot description, xacro)
@@ -27,7 +27,7 @@
   <xacro:property name="laser_h" value="0.06" />
   <xacro:property name="laser_x" value="0.03" />
-  <xacro:property name="laser_z" value="0.0787" />
+  <xacro:property name="laser_z" value="0.0094" />
   <joint name="laser_joint" type="fixed">
-    <origin xyz="${laser_x} 0 ${laser_z}" rpy="0 0 ${radians(-90)}"/>
+    <origin xyz="${laser_x} 0 ${laser_z}" rpy="${radians(180)} 0 ${radians(90)}"/>
     <parent link="base_link"/>
     <child link="base_laser_link"/>

Commit message: fix: robot size

File: urdf/minibot_light_01.xacro (robot description, xacro)
@@ -1,7 +1,7 @@
 <?xml version="1.0"?>
 <robot xmlns:xacro="http://www.ros.org/wiki/xacro" name="minibot_light_01">
-  <xacro:property name="body_d" value="0.24" />
-  <xacro:property name="body_w" value="0.24" />
-  <xacro:property name="body_h" value="0.158" />
+  <xacro:property name="body_d" value="0.23" />
+  <xacro:property name="body_w" value="0.23" />
+  <xacro:property name="body_h" value="0.132" />
   <xacro:property name="body_offset_x" value="-0.05" />
   <xacro:property name="body_offset_z" value="${body_h/2}" />

Commit message: add: xacro for gazebo

File: urdf/minibot_light_01.xacro (robot description, xacro)
@@ -1,20 +1,38 @@
 <?xml version="1.0"?>
 <robot xmlns:xacro="http://www.ros.org/wiki/xacro" name="minibot_light_01">
-  <xacro:property name="body_d" value="0.23" />
-  <xacro:property name="body_w" value="0.23" />
-  <xacro:property name="body_h" value="0.132" />
+  <!-- https://en.wikipedia.org/wiki/List_of_moments_of_inertia -->
+  <xacro:macro name="cylinder_inertia" params="m r h">
+    <inertia ixx="${m*(3*r*r+h*h)/12}" ixy = "0" ixz = "0" iyy="${m*(3*r*r+h*h)/12}" iyz = "0" izz="${m*r*r/2}" />
+  </xacro:macro>
+  <xacro:macro name="box_inertia" params="m x y z">
+    <inertia ixx="${m*(y*y+z*z)/12}" ixy = "0" ixz = "0" iyy="${m*(x*x+z*z)/12}" iyz = "0" izz="${m*(x*x+z*z)/12}" />
+  </xacro:macro>
+  <xacro:macro name="sphere_inertia" params="m r">
+    <inertia ixx="${2*m*r*r/5}" ixy = "0" ixz = "0" iyy="${2*m*r*r/5}" iyz = "0" izz="${2*m*r*r/5}" />
+  </xacro:macro>
+  <link name="base_link"/>
+  <xacro:property name="body_space" value="0.0195" />
+  <xacro:property name="body_size_x" value="0.23" />
+  <xacro:property name="body_size_y" value="0.23" />
+  <xacro:property name="body_size_z" value="${0.132 - body_space}" />
   <xacro:property name="body_offset_x" value="-0.05" />
-  <xacro:property name="body_offset_z" value="${body_h/2}" />
-  <link name="base_link">
+  <xacro:property name="body_offset_z" value="${body_space + body_size_z/2}" />
+  <xacro:property name="body_mass" value="1.0" />
+  <joint name="body_joint" type="fixed">
+    <origin rpy="0 0 0" xyz="${body_offset_x} 0 ${body_offset_z}"/>
+    <parent link="base_link"/>
+    <child link="body_link"/>
+  </joint>
+  <link name="body_link">
     <collision>
-      <origin rpy="0 0 0" xyz="${body_offset_x} 0 ${body_offset_z}"/>
+      <origin rpy="0 0 0" xyz="0 0 0"/>
       <geometry>
-        <box size="${body_d} ${body_w} ${body_h}"/>
+        <box size="${body_size_x} ${body_size_y} ${body_size_z}"/>
       </geometry>
     </collision>
     <visual>
-      <origin rpy="0 0 0" xyz="${body_offset_x} 0 ${body_offset_z}"/>
+      <origin rpy="0 0 0" xyz="0 0 0"/>
       <geometry>
-        <box size="${body_d} ${body_w} ${body_h}"/>
+        <box size="${body_size_x} ${body_size_y} ${body_size_z}"/>
       </geometry>
       <material name="vehicle_mat">
@@ -22,10 +40,15 @@
       </material>
     </visual>
+    <inertial>
+      <origin rpy="0 0 0" xyz="0 0 0"/>
+      <mass value="${body_mass}"/>
+      <xacro:box_inertia m="${body_mass}" x="${body_size_x}" y="${body_size_y}" z="${body_size_z}"/>
+    </inertial>
   </link>
-  <xacro:property name="laser_d" value="0.06" />
-  <xacro:property name="laser_w" value="0.06" />
-  <xacro:property name="laser_h" value="0.06" />
+  <xacro:property name="laser_radius" value="0.0328" />
+  <xacro:property name="laser_size_z" value="0.0352" />
   <xacro:property name="laser_x" value="0.03" />
   <xacro:property name="laser_z" value="0.0787" />
+  <xacro:property name="laser_mass" value="0.180" />
   <joint name="laser_joint" type="fixed">
     <origin xyz="${laser_x} 0 ${laser_z}" rpy="0 0 ${radians(-90)}"/>
@@ -37,5 +60,5 @@
       <origin rpy="0 0 0" xyz="0 0 0"/>
       <geometry>
-        <box size="${laser_d} ${laser_w} ${laser_h}"/>
+        <cylinder radius="${laser_radius}" length="${laser_size_z}"/>
       </geometry>
     </collision>
@@ -43,10 +66,15 @@
       <origin rpy="0 0 0" xyz="0 0 0"/>
       <geometry>
-        <box size="${laser_d} ${laser_w} ${laser_h}"/>
+        <cylinder radius="${laser_radius}" length="${laser_size_z}"/>
       </geometry>
       <material name="laser_mat">
-        <color rgba="0.0 0.0 0.0 0.8"/>
+        <color rgba="0.0 0.0 1.0 0.8"/>
       </material>
     </visual>
+    <inertial>
+      <origin rpy="0 0 0" xyz="0 0 0"/>
+      <mass value="${laser_mass}"/>
+      <xacro:cylinder_inertia m="${laser_mass}" r="${laser_radius}" h="${laser_size_z}"/>
+    </inertial>
   </link>
 </robot>

Commit message: fix: laser height and size

File: urdf/minibot_light_01.xacro (robot description, xacro)
@@ -3,12 +3,21 @@
   <!-- https://en.wikipedia.org/wiki/List_of_moments_of_inertia -->
   <xacro:macro name="cylinder_inertia" params="m r h">
+    <mass value="${m}"/>
     <inertia ixx="${m*(3*r*r+h*h)/12}" ixy = "0" ixz = "0" iyy="${m*(3*r*r+h*h)/12}" iyz = "0" izz="${m*r*r/2}" />
   </xacro:macro>
   <xacro:macro name="box_inertia" params="m x y z">
+    <mass value="${m}"/>
     <inertia ixx="${m*(y*y+z*z)/12}" ixy = "0" ixz = "0" iyy="${m*(x*x+z*z)/12}" iyz = "0" izz="${m*(x*x+z*z)/12}" />
   </xacro:macro>
   <xacro:macro name="sphere_inertia" params="m r">
+    <mass value="${m}"/>
     <inertia ixx="${2*m*r*r/5}" ixy = "0" ixz = "0" iyy="${2*m*r*r/5}" iyz = "0" izz="${2*m*r*r/5}" />
   </xacro:macro>
+  <material name="vehicle_mat">
+    <color rgba="1.0 0.0 0.0 0.5"/>
+  </material>
+  <material name="laser_mat">
+    <color rgba="0.0 0.0 1.0 0.8"/>
+  </material>
   <link name="base_link"/>
   <xacro:property name="body_space" value="0.0195" />
@@ -16,9 +25,15 @@
   <xacro:property name="body_size_y" value="0.23" />
   <xacro:property name="body_size_z" value="${0.132 - body_space}" />
-  <xacro:property name="body_offset_x" value="-0.05" />
-  <xacro:property name="body_offset_z" value="${body_space + body_size_z/2}" />
+  <!-- 0.1125 -->
+  <xacro:property name="body_x" value="-0.05" />
+  <xacro:property name="body_z" value="${body_space + body_size_z/2}" />
+  <!-- 0.07575 -->
   <xacro:property name="body_mass" value="1.0" />
+  <xacro:property name="body_panel_thickness" value="0.0055" />
+  <xacro:property name="body_panel_1_z" value="${-body_size_z/2 + body_panel_thickness/2}" />
+  <xacro:property name="body_panel_2_z" value="${body_panel_1_z + 0.05050}" />
+  <xacro:property name="body_panel_3_z" value="${body_panel_2_z + 0.05650}" />
   <joint name="body_joint" type="fixed">
-    <origin rpy="0 0 0" xyz="${body_offset_x} 0 ${body_offset_z}"/>
+    <origin rpy="0 0 0" xyz="${body_x} 0 ${body_z}"/>
     <parent link="base_link"/>
     <child link="body_link"/>
@@ -32,22 +47,38 @@
     </collision>
     <visual>
-      <origin rpy="0 0 0" xyz="0 0 0"/>
+      <origin rpy="0 0 0" xyz="0 0 ${body_panel_1_z}"/>
       <geometry>
-        <box size="${body_size_x} ${body_size_y} ${body_size_z}"/>
+        <box size="${body_size_x} ${body_size_y} ${body_panel_thickness}"/>
       </geometry>
-      <material name="vehicle_mat">
-        <color rgba="1.0 0.0 0.0 0.5"/>
-      </material>
+      <material name="vehicle_mat"/>
+    </visual>
+    <visual>
+      <origin rpy="0 0 0" xyz="0 0 ${body_panel_2_z}"/>
+      <geometry>
+        <box size="${body_size_x} ${body_size_y} ${body_panel_thickness}"/>
+      </geometry>
+      <material name="vehicle_mat"/>
+    </visual>
+    <visual>
+      <origin rpy="0 0 0" xyz="0 0 ${body_panel_3_z}"/>
+      <geometry>
+        <box size="${body_size_x} ${body_size_y} ${body_panel_thickness}"/>
+      </geometry>
+      <material name="vehicle_mat"/>
     </visual>
     <inertial>
       <origin rpy="0 0 0" xyz="0 0 0"/>
-      <mass value="${body_mass}"/>
       <xacro:box_inertia m="${body_mass}" x="${body_size_x}" y="${body_size_y}" z="${body_size_z}"/>
     </inertial>
   </link>
+  <gazebo reference="body_link">
+    <material>Gazebo/Red</material>
+    <mu1>0.05</mu1>
+    <mu2>0.05</mu2>
+  </gazebo>
   <xacro:property name="laser_radius" value="0.0328" />
   <xacro:property name="laser_size_z" value="0.0352" />
   <xacro:property name="laser_x" value="0.03" />
-  <xacro:property name="laser_z" value="0.0787" />
+  <xacro:property name="laser_z" value="${0.025 + laser_size_z/2}" />
   <xacro:property name="laser_mass" value="0.180" />
   <joint name="laser_joint" type="fixed">
@@ -68,13 +99,15 @@
         <cylinder radius="${laser_radius}" length="${laser_size_z}"/>
       </geometry>
-      <material name="laser_mat">
-        <color rgba="0.0 0.0 1.0 0.8"/>
-      </material>
+      <material name="laser_mat"/>
     </visual>
     <inertial>
       <origin rpy="0 0 0" xyz="0 0 0"/>
-      <mass value="${laser_mass}"/>
       <xacro:cylinder_inertia m="${laser_mass}" r="${laser_radius}" h="${laser_size_z}"/>
     </inertial>
   </link>
+  <gazebo reference="base_laser_link">
+    <material>Gazebo/Blue</material>
+    <mu1>0.05</mu1>
+    <mu2>0.05</mu2>
+  </gazebo>
 </robot>

Commit message: fix: sliding gazebo simulation

File: urdf/minibot_light_01.xacro (robot description, xacro)
@@ -24,4 +24,5 @@
   <xacro:property name="body_size_x" value="0.23" />
   <xacro:property name="body_size_y" value="0.23" />
+  <xacro:property name="body_collision_y" value="0.15" />
   <xacro:property name="body_size_z" value="${0.132 - body_space}" />
   <!-- 0.1125 -->
@@ -43,5 +44,5 @@
       <origin rpy="0 0 0" xyz="0 0 0"/>
       <geometry>
-        <box size="${body_size_x} ${body_size_y} ${body_size_z}"/>
+        <box size="${body_size_x} ${body_collision_y} ${body_size_z}"/>
       </geometry>
     </collision>
@@ -69,5 +70,5 @@
     <inertial>
       <origin rpy="0 0 0" xyz="0 0 0"/>
-      <xacro:box_inertia m="${body_mass}" x="${body_size_x}" y="${body_size_y}" z="${body_size_z}"/>
+      <xacro:box_inertia m="${body_mass}" x="${body_size_x}" y="${body_collision_y}" z="${body_size_z}"/>
     </inertial>
   </link>

File: urdf/minibot_light_01_gazebo.xacro (robot description, xacro)
@@ -40,8 +40,8 @@
   <xacro:property name="wheel_radius" value="0.03" />
   <xacro:property name="wheel_thickness" value="0.008" />
-  <xacro:property name="wheel_mass" value="0.011" />
+  <xacro:property name="wheel_mass" value="0.11" />
   <xacro:property name="wheel_damping" value="0.1" />
   <xacro:property name="wheel_friction" value="100" />
-  <xacro:property name="wheel_mu" value="2.5" />
+  <xacro:property name="wheel_mu" value="25" />
   <xacro:macro name="wheel_joint" params="prefix xyz rpy dumping friction">
     <joint name="${prefix}_wheel_joint" type="continuous">

Commit message: add: camera for gazebo

File: urdf/minibot_light_01.xacro (robot description, xacro)
@@ -20,4 +20,7 @@
     <color rgba="0.0 0.0 1.0 0.8"/>
   </material>
+  <material name="camera_mat">
+    <color rgba="0.0 1.0 0.0 0.8"/>
+  </material>
   <link name="base_link"/>
   <xacro:property name="body_space" value="0.0195" />
@@ -25,8 +28,7 @@
   <xacro:property name="body_size_y" value="0.23" />
   <xacro:property name="body_collision_y" value="0.15" />
-  <xacro:property name="body_size_z" value="${0.132 - body_space}" />
-  <!-- 0.1125 -->
+  <xacro:property name="body_size_z" value="0.1125" />
   <xacro:property name="body_x" value="-0.05" />
-  <xacro:property name="body_z" value="${body_space + body_size_z/2}" />
+  <xacro:property name="body_z" value="${body_space + body_size_z / 2}" />
   <!-- 0.07575 -->
   <xacro:property name="body_mass" value="1.0" />
@@ -54,5 +56,5 @@
       <material name="vehicle_mat"/>
     </visual>
-    <visual>
+    <!--visual>
       <origin rpy="0 0 0" xyz="0 0 ${body_panel_2_z}"/>
       <geometry>
@@ -67,5 +69,5 @@
       </geometry>
       <material name="vehicle_mat"/>
-    </visual>
+    </visual-->
     <inertial>
       <origin rpy="0 0 0" xyz="0 0 0"/>
@@ -112,3 +114,38 @@
     <mu2>0.05</mu2>
   </gazebo>
+  <xacro:property name="camera_size_x" value="0.006" />
+  <xacro:property name="camera_size_y" value="0.024" />
+  <xacro:property name="camera_size_z" value="0.024" />
+  <xacro:property name="camera_x" value="0.0289" />
+  <xacro:property name="camera_z" value="0.10125" />
+  <xacro:property name="camera_mass" value="0.010" />
+  <joint name="camera_joint" type="fixed">
+    <origin xyz="${camera_x} 0 ${camera_z}" rpy="0 0 0"/>
+    <parent link="base_link"/>
+    <child link="camera_link"/>
+  </joint>
+  <link name="camera_link">
+    <collision>
+      <origin rpy="0 0 0" xyz="0 0 0"/>
+      <geometry>
+        <box size="${camera_size_x} ${camera_size_y} ${camera_size_z}"/>
+      </geometry>
+    </collision>
+    <visual>
+      <origin rpy="0 0 0" xyz="0 0 0"/>
+      <geometry>
+        <box size="${camera_size_x} ${camera_size_y} ${camera_size_z}"/>
+      </geometry>
+      <material name="camera_mat"/>
+    </visual>
+    <inertial>
+      <origin rpy="0 0 0" xyz="0 0 0"/>
+      <xacro:box_inertia m="${camera_mass}" x="${camera_size_x}" y="${camera_size_y}" z="${camera_size_z}"/>
+    </inertial>
+  </link>
+  <gazebo reference="camera_link">
+    <material>Gazebo/Green</material>
+    <mu1>0.05</mu1>
+    <mu2>0.05</mu2>
+  </gazebo>
 </robot>

File: urdf/minibot_light_01_gazebo.xacro (robot description, xacro)
@@ -41,4 +41,5 @@
   <xacro:property name="wheel_thickness" value="0.008" />
   <xacro:property name="wheel_mass" value="0.11" />
+  <!--0.011-->
   <xacro:property name="wheel_damping" value="0.1" />
   <xacro:property name="wheel_friction" value="100" />
@@ -136,3 +137,39 @@
     </sensor>
   </gazebo>
+  <gazebo reference="camera_link">
+    <sensor type="camera" name="IMX219_D160">
+      <update_rate>30.0</update_rate>
+      <camera name="head">
+        <horizontal_fov>2.7074661906676</horizontal_fov>
+        <image>
+          <width>1280</width>
+          <height>720</height>
+          <format>R8G8B8</format>
+        </image>
+        <clip>
+          <near>0.05</near>
+          <far>300</far>
+        </clip>
+        <noise>
+          <type>gaussian</type>
+          <mean>0.0</mean>
+          <stddev>0.007</stddev>
+        </noise>
+      </camera>
+      <plugin name="camera_controller" filename="libgazebo_ros_camera.so">
+        <alwaysOn>true</alwaysOn>
+        <updateRate>0.0</updateRate>
+        <cameraName>video_source</cameraName>
+        <imageTopicName>raw</imageTopicName>
+        <cameraInfoTopicName>camera_info</cameraInfoTopicName>
+        <frameName>camera_link</frameName>
+        <hackBaseline>0.07</hackBaseline>
+        <distortionK1>0.0</distortionK1>
+        <distortionK2>0.0</distortionK2>
+        <distortionK3>0.0</distortionK3>
+        <distortionT1>0.0</distortionT1>
+        <distortionT2>0.0</distortionT2>
+      </plugin>
+    </sensor>
+  </gazebo>
 </robot>
